File: ftdi_debugger/hw/kicad/wasp1_ft2232h_debugger_revA/04_target_io.kicad_sch (KiCad schematic)
At the start: 16 parts, among them J2 WASP1 TARGET

Commit message: Harden FTDI manufacturing release package
Parts:
- TP1, TP2, TP3, TP4, TP5, TP6, TP7, TP8: now left out of the parts list
Changed lines of the file:
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@@
   )
   (symbol (lib_id "wasp1:TestPoint") (at 54.61 190.5 0) (unit 1)
-    (in_bom yes) (on_board yes) (dnp no)
+    (in_bom no) (on_board yes) (dnp no)
     (property "Reference" "TP1" (id 0) (at 44.45 180.34 0)
       (effects (font (size 1.27 1.27)))
@@
   )
   (symbol (lib_id "wasp1:TestPoint") (at 134.62 190.5 0) (unit 1)
-    (in_bom yes) (on_board yes) (dnp no)
+    (in_bom no) (on_board yes) (dnp no)
     (property "Reference" "TP2" (id 0) (at 124.46000000000001 180.34 0)
       (effects (font (size 1.27 1.27)))
@@
   )
   (symbol (lib_id "wasp1:TestPoint") (at 214.63 190.5 0) (unit 1)
-    (in_bom yes) (on_board yes) (dnp no)
+    (in_bom no) (on_board yes) (dnp no)
     (property "Reference" "TP3" (id 0) (at 204.47 180.34 0)
       (effects (font (size 1.27 1.27)))
@@
   )
   (symbol (lib_id "wasp1:TestPoint") (at 294.64 190.5 0) (unit 1)
-    (in_bom yes) (on_board yes) (dnp no)
+    (in_bom no) (on_board yes) (dnp no)
     (property "Reference" "TP4" (id 0) (at 284.47999999999996 180.34 0)
       (effects (font (size 1.27 1.27)))
@@
   )
   (symbol (lib_id "wasp1:TestPoint") (at 54.61 234.95000000000002 0) (unit 1)
-    (in_bom yes) (on_board yes) (dnp no)
+    (in_bom no) (on_board yes) (dnp no)
     (property "Reference" "TP5" (id 0) (at 44.45 224.79000000000002 0)
       (effects (font (size 1.27 1.27)))
@@
   )
   (symbol (lib_id "wasp1:TestPoint") (at 134.62 234.95000000000002 0) (unit 1)
-    (in_bom yes) (on_board yes) (dnp no)
+    (in_bom no) (on_board yes) (dnp no)
     (property "Reference" "TP6" (id 0) (at 124.46000000000001 224.79000000000002 0)
       (effects (font (size 1.27 1.27)))
@@
   )
   (symbol (lib_id "wasp1:TestPoint") (at 214.63 234.95000000000002 0) (unit 1)
-    (in_bom yes) (on_board yes) (dnp no)
+    (in_bom no) (on_board yes) (dnp no)
     (property "Reference" "TP7" (id 0) (at 204.47 224.79000000000002 0)
       (effects (font (size 1.27 1.27)))
@@
   )
   (symbol (lib_id "wasp1:TestPoint") (at 294.64 234.95000000000002 0) (unit 1)
-    (in_bom yes) (on_board yes) (dnp no)
+    (in_bom no) (on_board yes) (dnp no)
     (property "Reference" "TP8" (id 0) (at 284.47999999999996 224.79000000000002 0)
       (effects (font (size 1.27 1.27)))
